File: hardware/PCB/Hail_Mary.kicad_sch (KiCad schematic)
At the start: 0 parts

Commit message: PCB Footprints assigned and Layout added
Parts:
- added D1: LED, LED_THT:LED_D5.0mm, symbol Device:LED
- added J1: MPU6050, Connector_PinHeader_1.00mm:PinHeader_1x08_P1.00mm_Vertical, symbol Connector:Conn_01x08_Pin
- added J2: bmp280, Connector_PinHeader_1.00mm:PinHeader_1x06_P1.00mm_Vertical, symbol Connector:Conn_01x06_Pin
- added J3: ins_219, Connector_PinHeader_1.00mm:PinHeader_1x06_P1.00mm_Vertical, symbol Connector:Conn_01x06_Pin
- added J4: neo6m, Connector_PinHeader_1.00mm:PinHeader_1x04_P1.00mm_Vertical, symbol Connector:Conn_01x04_Pin
- added J5: proximity, Connector_PinHeader_1.00mm:PinHeader_1x03_P1.00mm_Vertical, symbol Connector:Conn_01x03_Pin
- added J6: impact, Connector_PinHeader_1.00mm:PinHeader_1x03_P1.00mm_Vertical, symbol Connector:Conn_01x03_Pin
- added R1: R, Resistor_THT:R_Axial_DIN0207_L6.3mm_D2.5mm_P10.16mm_Horizontal, symbol Device:R
- added SW1, SW2: SW_Push, Button_Switch_THT:SW_PUSH_6mm_H4.3mm, symbol Switch:SW_Push
- added U1: ESP32-C3-DevKitM-1, RF_Module:ESP32-C3-DevKitM-1, symbol RF_Module:ESP32-C3-DevKitM-1
Connections:
- new net: D1.2 (A), R1.2
- new net +5V: J4.1 (Pin_1), U1.13 (5V), U1.14 (5V)
- new net 3.3v: J1.1 (Pin_1), J2.1 (Pin_1), J3.1 (Pin_1), J5.1 (Pin_1), J6.1 (Pin_1), U1.2 (3V3), U1.3 (3V3)
- new net GND: D1.1 (K), J1.2 (Pin_2), J2.2 (Pin_2), J3.2 (Pin_2), J4.4 (Pin_4), J5.2 (Pin_2), J6.2 (Pin_2), SW1.1, SW2.1, U1.1 (GND), U1.12 (GND), U1.15 (GND), U1.16 (GND), U1.19 (GND), U1.24 (GND), U1.27 (GND), U1.30 (GND), U1.6 (GND), U1.8 (GND)
- new net ir_sensor: J5.3 (Pin_3), U1.9 (IO0)
- new net led: R1.1, U1.18 (IO18)
- new net master_button: SW1.2, U1.5 (IO3)
- new net nav_button: SW2.2, U1.11 (IO10)
- new net rx: J4.3 (Pin_3), U1.22 (IO6)
- new net scl: J1.3 (Pin_3), J2.3 (Pin_3), J3.3 (Pin_3), U1.21 (IO5)
- new net sda: J1.4 (Pin_4), J2.4 (Pin_4), J3.4 (Pin_4), U1.20 (IO4)
- new net sw_420: J6.3 (Pin_3), U1.10 (IO1)
- new net tx: J4.2 (Pin_2), U1.23 (IO7)
- no-connect marks 0 -> 15
